File: MoonLander_Sensors.sch (KiCad schematic (older format))
At the start: 2 parts

Commit message: schematic nearing prototype - time for some layout
Parts:
- added C? (x2): 0.1uF, symbol C
- added R?: 100k, symbol R
Connections:
- net GND: now also IC?.2 (GND), IC?.B2 (GND), IC?.C1 (ADR0), IC?.D1 (ADR1), C?.2, C?.2
- net I2C0_SDA: now also R?.2
- net RH_PWR: now reaches IC?.B1 (VDD)
- net RH_PWR: now also C?.1
- net RH_DRDY: now reaches IC?.D2 (~DRDY)
- net RH_DRDY: now also R?.1
- net LUX_PWR: now reaches IC?.1 (VDD)
- net LUX_PWR: now also C?.1
Other:
- moved on the sheet: IC?
Changed lines of the file:
@@
 $Descr A4 11693 8268
 encoding utf-8
-Sheet 5 5
+Sheet 5 6
 Title ""
 Date ""
@@
 Comment4 ""
 $EndDescr
-Text HLabel 2350 2500 0    60   Input ~ 0
+Text HLabel 3150 2500 0    60   Input ~ 0
 I2C0_SCL
-Text HLabel 2350 2600 0    60   BiDi ~ 0
+Text HLabel 3150 2600 0    60   BiDi ~ 0
 I2C0_SDA
 $Comp
 L HDC1008 IC?
 U 1 1 5660A0C7
-P 4950 2700
-F 0 "IC?" H 4750 3050 60  0000 C CNN
-F 1 "HDC1008" H 5050 2350 60  0000 C CNN
-F 2 "" H 5150 2550 60  0000 C CNN
-F 3 "" H 5150 2550 60  0000 C CNN
-	1    4950 2700
+P 5750 2700
+F 0 "IC?" H 5550 3050 60  0000 C CNN
+F 1 "HDC1008" H 5850 2350 60  0000 C CNN
+F 2 "" H 5950 2550 60  0000 C CNN
+F 3 "" H 5950 2550 60  0000 C CNN
+	1    5750 2700
 	1    0    0    -1
 $EndComp
@@
 L TSL4531 IC?
 U 1 1 5660A13A
-P 4950 4450
-F 0 "IC?" H 4800 4650 60  0000 C CNN
-F 1 "TSL4531" H 5000 4250 60  0000 C CNN
-F 2 "" H 5050 4350 60  0000 C CNN
-F 3 "" H 5050 4350 60  0000 C CNN
-	1    4950 4450
-	1    0    0    -1
-$EndComp
-Wire Wire Line
-	2350 2500 2650 2500
-Wire Wire Line
-	2650 2500 4450 2500
-Wire Wire Line
-	4450 2600 2550 2600
-Wire Wire Line
-	2550 2600 2350 2600
-Wire Wire Line
-	2650 2500 2650 4400
-Wire Wire Line
-	2650 4400 4500 4400
-Connection ~ 2650 2500
-Wire Wire Line
-	2550 2600 2550 4500
-Wire Wire Line
-	2550 4500 4500 4500
-Connection ~ 2550 2600
-$Comp
-L VCC #PWR?
-U 1 1 5660A200
-P 5550 4300
-F 0 "#PWR?" H 5550 4150 50  0001 C CNN
-F 1 "VCC" H 5550 4450 50  0000 C CNN
-F 2 "" H 5550 4300 50  0000 C CNN
-F 3 "" H 5550 4300 50  0000 C CNN
-	1    5550 4300
+P 5750 4450
+F 0 "IC?" H 5600 4650 60  0000 C CNN
+F 1 "TSL4531" H 5800 4250 60  0000 C CNN
+F 2 "" H 5850 4350 60  0000 C CNN
+F 3 "" H 5850 4350 60  0000 C CNN
+	1    5750 4450
 	1    0    0    -1
 $EndComp
@@
 L GND #PWR?
 U 1 1 5660A218
-P 5550 4600
-F 0 "#PWR?" H 5550 4350 50  0001 C CNN
-F 1 "GND" H 5550 4450 50  0000 C CNN
-F 2 "" H 5550 4600 50  0000 C CNN
-F 3 "" H 5550 4600 50  0000 C CNN
-	1    5550 4600
+P 6650 4800
+F 0 "#PWR?" H 6650 4550 50  0001 C CNN
+F 1 "GND" H 6650 4650 50  0000 C CNN
+F 2 "" H 6650 4800 50  0000 C CNN
+F 3 "" H 6650 4800 50  0000 C CNN
+	1    6650 4800
 	1    0    0    -1
 $EndComp
+$Comp
+L C C?
+U 1 1 56601857
+P 6650 4450
+F 0 "C?" H 6675 4550 50  0000 L CNN
+F 1 "0.1uF" H 6675 4350 50  0000 L CNN
+F 2 "" H 6688 4300 50  0000 C CNN
+F 3 "" H 6650 4450 50  0000 C CNN
+	1    6650 4450
+	1    0    0    -1
+$EndComp
+$Comp
+L GND #PWR?
+U 1 1 56601998
+P 6850 3100
+F 0 "#PWR?" H 6850 2850 50  0001 C CNN
+F 1 "GND" H 6850 2950 50  0000 C CNN
+F 2 "" H 6850 3100 50  0000 C CNN
+F 3 "" H 6850 3100 50  0000 C CNN
+	1    6850 3100
+	1    0    0    -1
+$EndComp
+$Comp
+L C C?
+U 1 1 5660199E
+P 6850 2750
+F 0 "C?" H 6875 2850 50  0000 L CNN
+F 1 "0.1uF" H 6875 2650 50  0000 L CNN
+F 2 "" H 6888 2600 50  0000 C CNN
+F 3 "" H 6850 2750 50  0000 C CNN
+	1    6850 2750
+	1    0    0    -1
+$EndComp
+Wire Wire Line
+	3150 2500 5250 2500
+Wire Wire Line
+	3150 2600 5250 2600
+Wire Wire Line
+	3450 2500 3450 4400
+Wire Wire Line
+	3450 4400 5300 4400
+Connection ~ 3450 2500
+Wire Wire Line
+	3350 2600 3350 4500
+Wire Wire Line
+	3350 4500 5300 4500
+Connection ~ 3350 2600
+Wire Wire Line
+	6200 4400 6350 4400
+Wire Wire Line
+	6350 4400 6350 4200
+Wire Wire Line
+	6650 4200 6650 4300
+Connection ~ 6650 4200
+Wire Wire Line
+	6200 4500 6350 4500
+Wire Wire Line
+	6350 4500 6350 4700
+Wire Wire Line
+	6350 4700 6650 4700
+Wire Wire Line
+	6650 4600 6650 4800
+Connection ~ 6650 4700
+Wire Wire Line
+	6850 2500 6850 2600
+Connection ~ 6850 2500
+Wire Wire Line
+	6450 3000 6850 3000
+Wire Wire Line
+	6850 2900 6850 3100
+Connection ~ 6850 3000
+Wire Wire Line
+	6250 2500 7250 2500
+Wire Wire Line
+	6350 4200 7250 4200
+Wire Wire Line
+	6250 2650 6450 2650
+Wire Wire Line
+	6450 2650 6450 3000
+Wire Wire Line
+	6450 2900 6250 2900
+Wire Wire Line
+	6250 2750 6450 2750
+Connection ~ 6450 2750
+Connection ~ 6450 2900
+Text HLabel 7250 2500 2    60   Input ~ 0
+RH_PWR
+$Comp
+L R R?
+U 1 1 56601E53
+P 4700 2750
+F 0 "R?" V 4780 2750 50  0000 C CNN
+F 1 "100k" V 4700 2750 50  0000 C CNN
+F 2 "" V 4630 2750 50  0000 C CNN
+F 3 "" H 4700 2750 50  0000 C CNN
+	1    4700 2750
+	0    1    1    0
+$EndComp
+Wire Wire Line
+	4550 2750 4450 2750
+Wire Wire Line
+	4450 2750 4450 2600
+Connection ~ 4450 2600
+Wire Wire Line
+	4850 2750 5250 2750
+Wire Wire Line
+	5000 2750 5000 3000
+Wire Wire Line
+	5000 3000 4650 3000
+Connection ~ 5000 2750
+Text HLabel 4650 3000 0    60   Output ~ 0
+RH_DRDY
+Text HLabel 7250 4200 2    60   Input ~ 0
+LUX_PWR
 $EndSCHEMATC

Commit message: first whack at layout - unrouted
Parts:
- C401, C402: renamed from C?; footprint (none) -> Capacitors_SMD:C_0402
- IC401: renamed from IC?; footprint (none) -> GrayCatLabs:TI-YPA0008
- IC402: renamed from IC?; footprint (none) -> GrayCatLabs:TSL4531
- R401: renamed from R?; footprint (none) -> Resistors_SMD:R_0402
Connections:
- net I2C0_SDA: no longer R401.2
- new net VCC: R401.2
Changed lines of the file:
@@
 I2C0_SDA
 $Comp
-L HDC1008 IC?
+L HDC1008 IC401
 U 1 1 5660A0C7
 P 5750 2700
-F 0 "IC?" H 5550 3050 60  0000 C CNN
+F 0 "IC401" H 5550 3050 60  0000 C CNN
 F 1 "HDC1008" H 5850 2350 60  0000 C CNN
-F 2 "" H 5950 2550 60  0000 C CNN
+F 2 "GrayCatLabs:TI-YPA0008" H 5950 2550 60  0001 C CNN
 F 3 "" H 5950 2550 60  0000 C CNN
 	1    5750 2700
@@
 $EndComp
 $Comp
-L TSL4531 IC?
+L TSL4531 IC402
 U 1 1 5660A13A
 P 5750 4450
-F 0 "IC?" H 5600 4650 60  0000 C CNN
+F 0 "IC402" H 5600 4650 60  0000 C CNN
 F 1 "TSL4531" H 5800 4250 60  0000 C CNN
-F 2 "" H 5850 4350 60  0000 C CNN
+F 2 "GrayCatLabs:TSL4531" H 5850 4350 60  0001 C CNN
 F 3 "" H 5850 4350 60  0000 C CNN
 	1    5750 4450
@@
 $EndComp
 $Comp
-L GND #PWR?
+L GND #PWR019
 U 1 1 5660A218
 P 6650 4800
-F 0 "#PWR?" H 6650 4550 50  0001 C CNN
+F 0 "#PWR019" H 6650 4550 50  0001 C CNN
 F 1 "GND" H 6650 4650 50  0000 C CNN
 F 2 "" H 6650 4800 50  0000 C CNN
@@
 $EndComp
 $Comp
-L C C?
+L C C401
 U 1 1 56601857
 P 6650 4450
-F 0 "C?" H 6675 4550 50  0000 L CNN
+F 0 "C401" H 6675 4550 50  0000 L CNN
 F 1 "0.1uF" H 6675 4350 50  0000 L CNN
-F 2 "" H 6688 4300 50  0000 C CNN
+F 2 "Capacitors_SMD:C_0402" H 6688 4300 50  0001 C CNN
 F 3 "" H 6650 4450 50  0000 C CNN
 	1    6650 4450
@@
 $EndComp
 $Comp
-L GND #PWR?
+L GND #PWR020
 U 1 1 56601998
 P 6850 3100
-F 0 "#PWR?" H 6850 2850 50  0001 C CNN
+F 0 "#PWR020" H 6850 2850 50  0001 C CNN
 F 1 "GND" H 6850 2950 50  0000 C CNN
 F 2 "" H 6850 3100 50  0000 C CNN
@@
 $EndComp
 $Comp
-L C C?
+L C C402
 U 1 1 5660199E
 P 6850 2750
-F 0 "C?" H 6875 2850 50  0000 L CNN
+F 0 "C402" H 6875 2850 50  0000 L CNN
 F 1 "0.1uF" H 6875 2650 50  0000 L CNN
-F 2 "" H 6888 2600 50  0000 C CNN
+F 2 "Capacitors_SMD:C_0402" H 6888 2600 50  0001 C CNN
 F 3 "" H 6850 2750 50  0000 C CNN
 	1    6850 2750
@@
 RH_PWR
 $Comp
-L R R?
+L R R401
 U 1 1 56601E53
 P 4700 2750
-F 0 "R?" V 4780 2750 50  0000 C CNN
+F 0 "R401" V 4780 2750 50  0000 C CNN
 F 1 "100k" V 4700 2750 50  0000 C CNN
-F 2 "" V 4630 2750 50  0000 C CNN
+F 2 "Resistors_SMD:R_0402" V 4630 2750 50  0001 C CNN
 F 3 "" H 4700 2750 50  0000 C CNN
 	1    4700 2750
@@
 Wire Wire Line
 	4550 2750 4450 2750
-Wire Wire Line
-	4450 2750 4450 2600
-Connection ~ 4450 2600
 Wire Wire Line
 	4850 2750 5250 2750
@@
 Text HLabel 7250 4200 2    60   Input ~ 0
 LUX_PWR
+$Comp
+L VCC #PWR021
+U 1 1 56634F19
+P 4450 2750
+F 0 "#PWR021" H 4450 2600 50  0001 C CNN
+F 1 "VCC" H 4450 2900 50  0000 C CNN
+F 2 "" H 4450 2750 50  0000 C CNN
+F 3 "" H 4450 2750 50  0000 C CNN
+	1    4450 2750
+	0    -1   -1   0
+$EndComp
 $EndSCHEMATC
