File: MoonLander_CPU.sch (KiCad schematic (older format))
At the start: 13 parts

Commit message: schematic nearing prototype - time for some layout
Parts:
- added C? (x2): 0.1uF, symbol C
- added R? (x2): 100k, symbol R
Connections:
- net GND: now also C?.2, C?.2, R?.2
- net ISP_ENTRY: now also C?.1
- net PIO0_1 renamed LED_R
- net PIO0_24 renamed RH_PWR
- net PIO0_25 renamed RH_DRDY
- net PIO0_26 renamed LUX_PWR
- net PIO0_27 renamed LED_G
- net PIO0_28 renamed LED_B
- net PIO0_6_ADC_1 renamed PIO0_6/ADC_1
- net PIO0_7/ADC_0: no longer names the net of IC?.22 (PIO0_7/ADC_0)
- net PIO0_7/ADC_0: now also C?.1, R?.1, R?.2
- new net V_BAT: R?.1
Other:
- moved on the sheet: R?
Changed lines of the file:
@@
 $Descr A4 11693 8268
 encoding utf-8
-Sheet 4 5
+Sheet 6 6
 Title ""
 Date ""
@@
 	1    0    0    -1
 $EndComp
-Text HLabel 3100 4650 0    60   BiDi ~ 0
+Text HLabel 3100 4650 0    60   Input ~ 0
 ISP_RXD
 Wire Wire Line
-	3950 3250 3950 3450
+	3950 3250 3950 3350
+Wire Wire Line
+	3950 3350 3950 3450
 Wire Wire Line
 	3950 3450 4300 3450
@@
 	4300 3700 3950 3700
 Wire Wire Line
-	3950 3700 3950 3850
-Wire Wire Line
-	3350 3800 4300 3800
+	3950 3700 3950 3800
+Wire Wire Line
+	3950 3800 3950 3850
+Wire Wire Line
+	3350 3800 3750 3800
+Wire Wire Line
+	3750 3800 3950 3800
+Wire Wire Line
+	3950 3800 4300 3800
 Connection ~ 3950 3800
 Wire Wire Line
@@
 	6700 1550 6700 2050
 Wire Wire Line
-	6700 1050 6700 1250
-Wire Wire Line
-	6200 1150 6700 1150
+	6700 1050 6700 1150
+Wire Wire Line
+	6700 1150 6700 1250
+Wire Wire Line
+	6200 1150 6450 1150
+Wire Wire Line
+	6450 1150 6700 1150
 Wire Wire Line
 	6450 1150 6450 1250
@@
 	4500 2050 4600 2050
 Wire Wire Line
-	4500 1750 4500 2150
+	4500 1750 4500 1850
+Wire Wire Line
+	4500 1850 4500 2050
+Wire Wire Line
+	4500 2050 4500 2150
 Wire Wire Line
 	4600 1850 4500 1850
@@
 Connection ~ 3750 3800
 Wire Wire Line
-	3350 3350 4300 3350
+	3350 3350 3750 3350
+Wire Wire Line
+	3750 3350 3950 3350
+Wire Wire Line
+	3950 3350 4300 3350
 Wire Wire Line
 	4150 4150 4150 4300
 Wire Wire Line
-	3650 4150 4150 4150
+	3650 4150 3900 4150
+Wire Wire Line
+	3900 4150 4150 4150
 Wire Wire Line
 	3900 4150 3900 4200
@@
 	4150 4550 4150 4400
 Wire Wire Line
-	3650 4550 4150 4550
+	3650 4550 3900 4550
+Wire Wire Line
+	3900 4550 4150 4550
 Wire Wire Line
 	3900 4550 3900 4500
@@
 	3250 4200 3150 4200
 Wire Wire Line
-	3150 4200 3150 4500
+	3150 4200 3150 4350
+Wire Wire Line
+	3150 4350 3150 4500
 Wire Wire Line
 	3150 4500 3250 4500
@@
 	4300 4950 3350 4950
 Wire Wire Line
-	6900 3350 7750 3350
-Wire Wire Line
-	6900 3450 7750 3450
+	6900 3350 7150 3350
+Wire Wire Line
+	7150 3350 7750 3350
+Wire Wire Line
+	6900 3450 7400 3450
+Wire Wire Line
+	7400 3450 7750 3450
 Wire Wire Line
 	7400 3250 7400 3450
@@
 Connection ~ 7150 3350
 Wire Wire Line
-	7150 2750 7150 2950
+	7150 2750 7150 2850
+Wire Wire Line
+	7150 2850 7150 2950
 Wire Wire Line
 	7400 2850 7400 2950
@@
 	3100 4750 4300 4750
 Text HLabel 3100 4750 0    60   BiDi ~ 0
-PIO0_1
-Text HLabel 3100 5050 0    60   BiDi ~ 0
+LED_R
+Text HLabel 3100 5050 0    60   Output ~ 0
 ISP_TXD
 Text HLabel 3100 5150 0    60   BiDi ~ 0
-PIO0_6_ADC_1
-Text HLabel 3100 5250 0    60   BiDi ~ 0
-PIO0_7/ADC_0
+PIO0_6/ADC_1
 Wire Wire Line
 	3100 5150 4300 5150
 Wire Wire Line
-	4300 5250 3100 5250
+	1650 5250 2000 5250
+Wire Wire Line
+	2000 5250 4300 5250
 Text HLabel 7750 3650 2    60   BiDi ~ 0
 PIO0_13/ADC_10
@@
 Text HLabel 7750 4700 2    60   BiDi ~ 0
 PIO0_23/ADC_3
-Text HLabel 7750 4850 2    60   BiDi ~ 0
-PIO0_24
-Text HLabel 7750 4950 2    60   BiDi ~ 0
-PIO0_25
-Text HLabel 7750 5050 2    60   BiDi ~ 0
-PIO0_26
+Text HLabel 7750 4950 2    60   Input ~ 0
+RH_DRDY
+Text HLabel 7750 4850 2    60   Output ~ 0
+RH_PWR
+Text HLabel 7750 5050 2    60   Output ~ 0
+LUX_PWR
 Text HLabel 7750 5150 2    60   BiDi ~ 0
-PIO0_27
+LED_G
 Text HLabel 7750 5250 2    60   BiDi ~ 0
-PIO0_28
+LED_B
 Wire Wire Line
 	7750 5250 6900 5250
@@
 	6900 3550 9050 3550
 Wire Wire Line
-	8700 3550 8700 3350
+	9050 3550 9550 3550
+Wire Wire Line
+	9050 3350 9050 3550
+Wire Wire Line
+	9050 3550 9050 3700
 $Comp
 L R R?
 U 1 1 565F7CAC
-P 8700 3200
-F 0 "R?" V 8780 3200 50  0000 C CNN
-F 1 "100k" V 8700 3200 50  0000 C CNN
-F 2 "" V 8630 3200 50  0000 C CNN
-F 3 "" H 8700 3200 50  0000 C CNN
-	1    8700 3200
-	1    0    0    -1
-$EndComp
-Wire Wire Line
-	8700 2850 8700 3050
-Connection ~ 8700 3550
-Text HLabel 9050 3550 2    60   Input ~ 0
+P 9050 3200
+F 0 "R?" V 9130 3200 50  0000 C CNN
+F 1 "100k" V 9050 3200 50  0000 C CNN
+F 2 "" V 8980 3200 50  0000 C CNN
+F 3 "" H 9050 3200 50  0000 C CNN
+	1    9050 3200
+	1    0    0    -1
+$EndComp
+Wire Wire Line
+	9050 2850 9050 3050
+Connection ~ 9050 3550
+Text HLabel 9550 3550 2    60   Input ~ 0
 ISP_ENTRY
 Wire Wire Line
@@
 L VCC #PWR?
 U 1 1 565F82A6
-P 8700 2850
-F 0 "#PWR?" H 8700 2700 50  0001 C CNN
-F 1 "VCC" H 8700 3000 50  0000 C CNN
-F 2 "" H 8700 2850 50  0000 C CNN
-F 3 "" H 8700 2850 50  0000 C CNN
-	1    8700 2850
-	1    0    0    -1
-$EndComp
+P 9050 2850
+F 0 "#PWR?" H 9050 2700 50  0001 C CNN
+F 1 "VCC" H 9050 3000 50  0000 C CNN
+F 2 "" H 9050 2850 50  0000 C CNN
+F 3 "" H 9050 2850 50  0000 C CNN
+	1    9050 2850
+	1    0    0    -1
+$EndComp
+Text HLabel 1500 4700 0    60   Input ~ 0
+V_BAT
+$Comp
+L R R?
+U 1 1 565FF896
+P 1650 4950
+F 0 "R?" V 1730 4950 50  0000 C CNN
+F 1 "100k" V 1650 4950 50  0000 C CNN
+F 2 "" V 1580 4950 50  0000 C CNN
+F 3 "" H 1650 4950 50  0000 C CNN
+	1    1650 4950
+	1    0    0    -1
+$EndComp
+$Comp
+L R R?
+U 1 1 565FF90C
+P 1650 5550
+F 0 "R?" V 1730 5550 50  0000 C CNN
+F 1 "100k" V 1650 5550 50  0000 C CNN
+F 2 "" V 1580 5550 50  0000 C CNN
+F 3 "" H 1650 5550 50  0000 C CNN
+	1    1650 5550
+	1    0    0    -1
+$EndComp
+$Comp
+L GND #PWR?
+U 1 1 565FF956
+P 1650 5950
+F 0 "#PWR?" H 1650 5700 50  0001 C CNN
+F 1 "GND" H 1650 5800 50  0000 C CNN
+F 2 "" H 1650 5950 50  0000 C CNN
+F 3 "" H 1650 5950 50  0000 C CNN
+	1    1650 5950
+	1    0    0    -1
+$EndComp
+Wire Wire Line
+	1650 5700 1650 5850
+Wire Wire Line
+	1650 5850 1650 5950
+Wire Wire Line
+	1650 5100 1650 5250
+Wire Wire Line
+	1650 5250 1650 5400
+Connection ~ 1650 5250
+Wire Wire Line
+	1500 4700 1650 4700
+Wire Wire Line
+	1650 4700 1650 4800
+$Comp
+L C C?
+U 1 1 56600253
+P 2000 5550
+F 0 "C?" H 2025 5650 50  0000 L CNN
+F 1 "0.1uF" H 2025 5450 50  0000 L CNN
+F 2 "" H 2038 5400 50  0000 C CNN
+F 3 "" H 2000 5550 50  0000 C CNN
+	1    2000 5550
+	1    0    0    -1
+$EndComp
+Wire Wire Line
+	2000 5700 2000 5850
+Wire Wire Line
+	2000 5850 1650 5850
+Connection ~ 1650 5850
+Wire Wire Line
+	2000 5250 2000 5400
+Connection ~ 2000 5250
+$Comp
+L C C?
+U 1 1 56610699
+P 9050 3850
+F 0 "C?" H 9075 3950 50  0000 L CNN
+F 1 "0.1uF" H 9075 3750 50  0000 L CNN
+F 2 "" H 9088 3700 50  0000 C CNN
+F 3 "" H 9050 3850 50  0000 C CNN
+	1    9050 3850
+	1    0    0    -1
+$EndComp
+$Comp
+L GND #PWR?
+U 1 1 56610766
+P 9050 4100
+F 0 "#PWR?" H 9050 3850 50  0001 C CNN
+F 1 "GND" H 9050 3950 50  0000 C CNN
+F 2 "" H 9050 4100 50  0000 C CNN
+F 3 "" H 9050 4100 50  0000 C CNN
+	1    9050 4100
+	1    0    0    -1
+$EndComp
+Wire Wire Line
+	9050 4100 9050 4000
 $EndSCHEMATC

Commit message: first whack at layout - unrouted
Parts:
- removed C?: 0.1uF, symbol C
- added C605: 0.1uF, Capacitors_SMD:C_0402, symbol C
- C601, C602, C606: renamed from C?; footprint (none) -> Capacitors_SMD:C_0402
- C603, C604: renamed from C?; value C -> 18pF; footprint (none) -> Capacitors_SMD:C_0402
- IC601: renamed from IC?; footprint (none) -> Housings_DFN_QFN:QFN-32-1EP_5x5mm_Pitch0.5mm
- J601: renamed from J?; footprint (none) -> Pin_Headers:Pin_Header_Straight_2x05_Pitch1.27mm
- R601, R602, R603, R604, R605, R606, R607, R608: renamed from R?; footprint (none) -> Resistors_SMD:R_0402
- Y601: renamed from Y?; footprint (none) -> Crystals:crystal_FA238-TSX3225
Connections:
- net GND: now also C605.2
- net LED_B: now also IC601.11 (PIO0_27); no longer IC601.5 (PIO0_28/WKTCLKIN)
- net LED_G: now also IC601.16 (PIO0_1/ACMP_I2/CLKIN/TDI); no longer IC601.11 (PIO0_27)
- net LED_R: now also IC601.5 (PIO0_28/WKTCLKIN); no longer IC601.16 (PIO0_1/ACMP_I2/CLKIN/TDI)
- net RESET: now also C605.1
Other:
- moved on the sheet: C602

Commit message: simplified 2 layer version
Parts:
- renumbered C605 to C10, C603 to C11, C604 to C12, C602 to C13, C606 to C14, C601 to C9, IC601 to IC5, J601 to J1, R605 to R10, R606 to R11, R607 to R12, R608 to R13, R601 to R6, R602 to R7, R603 to R8, R604 to R9, Y601 to Y1
Connections:
- net LED_B: no longer names the net of IC5.11 (PIO0_27)
- net LED_G: no longer names the net of IC5.16 (PIO0_1/ACMP_I2/CLKIN/TDI)
- net LED_R renamed LED
- net LUX_PWR: no longer names the net of IC5.12 (PIO0_26)
- net PIO0_15: no longer names the net of IC5.15 (PIO0_15)
- net PIO0_16: no longer names the net of IC5.10 (PIO0_16)
- net RH_DRDY: no longer names the net of IC5.13 (PIO0_25)
- net RH_PWR: no longer names the net of IC5.14 (PIO0_24)
Changed lines of the file:
@@
 $Descr A4 11693 8268
 encoding utf-8
-Sheet 6 6
+Sheet 5 5
 Title ""
 Date ""
@@
 $EndDescr
 $Comp
-L LPC824M201JHI33 IC601
+L LPC824M201JHI33 IC5
 U 1 1 565F2D73
 P 5600 4300
-F 0 "IC601" H 4600 5400 60  0000 C CNN
+F 0 "IC5" H 4600 5400 60  0000 C CNN
 F 1 "LPC824M201JHI33" H 6250 3200 60  0000 C CNN
 F 2 "Housings_DFN_QFN:QFN-32-1EP_5x5mm_Pitch0.5mm" H 6100 5000 60  0001 C CNN
@@
 $EndComp
 $Comp
-L VCC #PWR026
+L VCC #PWR021
 U 1 1 565F2E16
 P 3950 3250
-F 0 "#PWR026" H 3950 3100 50  0001 C CNN
+F 0 "#PWR021" H 3950 3100 50  0001 C CNN
 F 1 "VCC" H 3950 3400 50  0000 C CNN
 F 2 "" H 3950 3250 50  0000 C CNN
@@
 $EndComp
 $Comp
-L GND #PWR027
+L GND #PWR022
 U 1 1 565F2E2E
 P 3950 3850
-F 0 "#PWR027" H 3950 3600 50  0001 C CNN
+F 0 "#PWR022" H 3950 3600 50  0001 C CNN
 F 1 "GND" H 3950 3700 50  0000 C CNN
 F 2 "" H 3950 3850 50  0000 C CNN
@@
 $EndComp
 $Comp
-L Cortex_JTAG/SWD_10 J601
+L Cortex_JTAG/SWD_10 J1
 U 1 1 565F3829
 P 5200 1850
-F 0 "J601" H 4900 2200 60  0000 C CNN
+F 0 "J1" H 4900 2200 60  0000 C CNN
 F 1 "Cortex_JTAG/SWD_10" H 5250 1500 60  0000 C CNN
 F 2 "Pin_Headers:Pin_Header_Straight_2x05_Pitch1.27mm" H 5100 1450 60  0001 C CNN
@@
 $EndComp
 $Comp
-L R R603
+L R R8
 U 1 1 565F395C
 P 6200 1400
-F 0 "R603" V 6280 1400 50  0000 C CNN
+F 0 "R8" V 6280 1400 50  0000 C CNN
 F 1 "10k" V 6200 1400 50  0000 C CNN
 F 2 "Resistors_SMD:R_0402" V 6130 1400 50  0001 C CNN
@@
 $EndComp
 $Comp
-L R R604
+L R R9
 U 1 1 565F39B6
 P 6450 1400
-F 0 "R604" V 6530 1400 50  0000 C CNN
+F 0 "R9" V 6530 1400 50  0000 C CNN
 F 1 "10k" V 6450 1400 50  0000 C CNN
 F 2 "Resistors_SMD:R_0402" V 6380 1400 50  0001 C CNN
@@
 SWDIO
 $Comp
-L R R605
+L R R10
 U 1 1 565F3AF6
 P 6700 1400
-F 0 "R605" V 6780 1400 50  0000 C CNN
+F 0 "R10" V 6780 1400 50  0000 C CNN
 F 1 "10k" V 6700 1400 50  0000 C CNN
 F 2 "Resistors_SMD:R_0402" V 6630 1400 50  0001 C CNN
@@
 $EndComp
 $Comp
-L VCC #PWR028
+L VCC #PWR023
 U 1 1 565F3B82
 P 6700 1050
-F 0 "#PWR028" H 6700 900 50  0001 C CNN
+F 0 "#PWR023" H 6700 900 50  0001 C CNN
 F 1 "VCC" H 6700 1200 50  0000 C CNN
 F 2 "" H 6700 1050 50  0000 C CNN
@@
 $EndComp
 $Comp
-L VCC #PWR029
+L VCC #PWR024
 U 1 1 565F3C33
 P 4500 1500
-F 0 "#PWR029" H 4500 1350 50  0001 C CNN
+F 0 "#PWR024" H 4500 1350 50  0001 C CNN
 F 1 "VCC" H 4500 1650 50  0000 C CNN
 F 2 "" H 4500 1500 50  0000 C CNN
@@
 $EndComp
 $Comp
-L GND #PWR030
+L GND #PWR025
 U 1 1 565F3C7E
 P 4500 2150
-F 0 "#PWR030" H 4500 1900 50  0001 C CNN
+F 0 "#PWR025" H 4500 1900 50  0001 C CNN
 F 1 "GND" H 4500 2000 50  0000 C CNN
 F 2 "" H 4500 2150 50  0000 C CNN
@@
 RESET
 $Comp
-L C C602
+L C C13
 U 1 1 565F4293
 P 3600 3600
-F 0 "C602" H 3625 3700 50  0000 L CNN
+F 0 "C13" H 3625 3700 50  0000 L CNN
 F 1 "0.1uF" H 3625 3500 50  0000 L CNN
 F 2 "Capacitors_SMD:C_0402" H 3638 3450 50  0001 C CNN
@@
 $EndComp
 $Comp
-L C C604
+L C C12
 U 1 1 565F47F2
 P 3400 4500
-F 0 "C604" H 3425 4600 50  0000 L CNN
+F 0 "C12" H 3425 4600 50  0000 L CNN
 F 1 "18pF" H 3425 4400 50  0000 L CNN
 F 2 "Capacitors_SMD:C_0402" H 3438 4350 50  0001 C CNN
@@
 $EndComp
 $Comp
-L C C603
+L C C11
 U 1 1 565F4825
 P 3400 4200
-F 0 "C603" H 3425 4300 50  0000 L CNN
+F 0 "C11" H 3425 4300 50  0000 L CNN
 F 1 "18pF" H 3425 4100 50  0000 L CNN
 F 2 "Capacitors_SMD:C_0402" H 3438 4050 50  0001 C CNN
@@
 $EndComp
 $Comp
-L Crystal Y601
+L Crystal Y1
 U 1 1 565F4A39
 P 3900 4350
-F 0 "Y601" H 3900 4500 50  0000 C CNN
+F 0 "Y1" H 3900 4500 50  0000 C CNN
 F 1 "Crystal" H 3900 4200 50  0000 C CNN
 F 2 "Crystals:crystal_FA238-TSX3225" H 3900 4350 50  0001 C CNN
@@
 $EndComp
 $Comp
-L GND #PWR031
+L GND #PWR026
 U 1 1 565F4D06
 P 3050 4350
-F 0 "#PWR031" H 3050 4100 50  0001 C CNN
+F 0 "#PWR026" H 3050 4100 50  0001 C CNN
 F 1 "GND" H 3050 4200 50  0000 C CNN
 F 2 "" H 3050 4350 50  0000 C CNN
@@
 SWCLK
 $Comp
-L R R606
+L R R11
 U 1 1 565F544F
 P 7150 3100
-F 0 "R606" V 7230 3100 50  0000 C CNN
+F 0 "R11" V 7230 3100 50  0000 C CNN
 F 1 "10k" V 7150 3100 50  0000 C CNN
 F 2 "Resistors_SMD:R_0402" V 7080 3100 50  0001 C CNN
@@
 $EndComp
 $Comp
-L R R607
+L R R12
 U 1 1 565F5541
 P 7400 3100
-F 0 "R607" V 7480 3100 50  0000 C CNN
+F 0 "R12" V 7480 3100 50  0000 C CNN
 F 1 "10k" V 7400 3100 50  0000 C CNN
 F 2 "Resistors_SMD:R_0402" V 7330 3100 50  0001 C CNN
@@
 I2C0_SDA
 $Comp
-L VCC #PWR032
+L VCC #PWR027
 U 1 1 565F57DE
 P 7150 2750
-F 0 "#PWR032" H 7150 2600 50  0001 C CNN
+F 0 "#PWR027" H 7150 2600 50  0001 C CNN
 F 1 "VCC" H 7150 2900 50  0000 C CNN
 F 2 "" H 7150 2750 50  0000 C CNN
@@
 Wire Wire Line
 	3100 4650 4300 4650
-Wire Wire Line
-	3100 4750 4300 4750
-Text HLabel 3100 4750 0    60   BiDi ~ 0
-LED_G
 Text HLabel 3100 5050 0    60   Output ~ 0
 ISP_TXD
@@
 Text HLabel 7750 3750 2    60   BiDi ~ 0
 PIO0_14/ADC_2
-Text HLabel 7750 3850 2    60   BiDi ~ 0
-PIO0_15
-Text HLabel 7750 4000 2    60   BiDi ~ 0
-PIO0_16
 Text HLabel 7750 4100 2    60   BiDi ~ 0
 PIO0_17/ADC_9
@@
 Text HLabel 7750 4700 2    60   BiDi ~ 0
 PIO0_23/ADC_3
-Text HLabel 7750 4950 2    60   Input ~ 0
-RH_DRDY
-Text HLabel 7750 4850 2    60   Output ~ 0
-RH_PWR
-Text HLabel 7750 5050 2    60   Output ~ 0
-LUX_PWR
-Text HLabel 7750 5150 2    60   BiDi ~ 0
-LED_B
-Text HLabel 7750 5250 2    60   BiDi ~ 0
-LED_R
+Text HLabel 7750 5250 2    60   Output ~ 0
+LED
 Wire Wire Line
 	7750 5250 6900 5250
 Wire Wire Line
-	6900 5150 7750 5150
-Wire Wire Line
-	7750 5050 6900 5050
-Wire Wire Line
-	6900 4950 7750 4950
-Wire Wire Line
-	7750 4850 6900 4850
-Wire Wire Line
 	6900 4700 7750 4700
 Wire Wire Line
@@
 	6900 4100 7750 4100
 Wire Wire Line
-	7750 4000 6900 4000
-Wire Wire Line
-	6900 3850 7750 3850
-Wire Wire Line
 	7750 3750 6900 3750
 Wire Wire Line
@@
 	9050 3350 9050 3700
 $Comp
-L R R608
+L R R13
 U 1 1 565F7CAC
 P 9050 3200
-F 0 "R608" V 9130 3200 50  0000 C CNN
+F 0 "R13" V 9130 3200 50  0000 C CNN
 F 1 "100k" V 9050 3200 50  0000 C CNN
 F 2 "Resistors_SMD:R_0402" V 8980 3200 50  0001 C CNN
@@
 	7400 2850 7150 2850
 $Comp
-L VCC #PWR033
+L VCC #PWR028
 U 1 1 565F82A6
 P 9050 2850
-F 0 "#PWR033" H 9050 2700 50  0001 C CNN
+F 0 "#PWR028" H 9050 2700 50  0001 C CNN
 F 1 "VCC" H 9050 3000 50  0000 C CNN
 F 2 "" H 9050 2850 50  0000 C CNN
@@
 V_BAT
 $Comp
-L R R601
+L R R6
 U 1 1 565FF896
 P 1650 4950
-F 0 "R601" V 1730 4950 50  0000 C CNN
+F 0 "R6" V 1730 4950 50  0000 C CNN
 F 1 "100k" V 1650 4950 50  0000 C CNN
 F 2 "Resistors_SMD:R_0402" V 1580 4950 50  0001 C CNN
@@
 $EndComp
 $Comp
-L R R602
+L R R7
 U 1 1 565FF90C
 P 1650 5550
-F 0 "R602" V 1730 5550 50  0000 C CNN
+F 0 "R7" V 1730 5550 50  0000 C CNN
 F 1 "100k" V 1650 5550 50  0000 C CNN
 F 2 "Resistors_SMD:R_0402" V 1580 5550 50  0001 C CNN
@@
 $EndComp
 $Comp
-L GND #PWR034
+L GND #PWR029
 U 1 1 565FF956
 P 1650 5950
-F 0 "#PWR034" H 1650 5700 50  0001 C CNN
+F 0 "#PWR029" H 1650 5700 50  0001 C CNN
 F 1 "GND" H 1650 5800 50  0000 C CNN
 F 2 "" H 1650 5950 50  0000 C CNN
@@
 	1650 4700 1650 4800
 $Comp
-L C C601
+L C C9
 U 1 1 56600253
 P 2000 5550
-F 0 "C601" H 2025 5650 50  0000 L CNN
+F 0 "C9" H 2025 5650 50  0000 L CNN
 F 1 "0.1uF" H 2025 5450 50  0000 L CNN
 F 2 "Capacitors_SMD:C_0402" H 2038 5400 50  0001 C CNN
@@
 Connection ~ 2000 5250
 $Comp
-L C C606
+L C C14
 U 1 1 56610699
 P 9050 3850
-F 0 "C606" H 9075 3950 50  0000 L CNN
+F 0 "C14" H 9075 3950 50  0000 L CNN
 F 1 "0.1uF" H 9075 3750 50  0000 L CNN
 F 2 "Capacitors_SMD:C_0402" H 9088 3700 50  0001 C CNN
@@
 $EndComp
 $Comp
-L GND #PWR035
+L GND #PWR030
 U 1 1 56610766
 P 9050 4100
-F 0 "#PWR035" H 9050 3850 50  0001 C CNN
+F 0 "#PWR030" H 9050 3850 50  0001 C CNN
 F 1 "GND" H 9050 3950 50  0000 C CNN
 F 2 "" H 9050 4100 50  0000 C CNN
@@
 	3600 3350 4300 3350
 $Comp
-L C C605
+L C C10
 U 1 1 566346FD
 P 2200 4300
-F 0 "C605" H 2225 4400 50  0000 L CNN
+F 0 "C10" H 2225 4400 50  0000 L CNN
 F 1 "0.1uF" H 2225 4200 50  0000 L CNN
 F 2 "Capacitors_SMD:C_0402" H 2238 4150 50  0001 C CNN
@@
 $EndComp
 $Comp
-L GND #PWR036
+L GND #PWR031
 U 1 1 56634895
 P 2200 4550
-F 0 "#PWR036" H 2200 4300 50  0001 C CNN
+F 0 "#PWR031" H 2200 4300 50  0001 C CNN
 F 1 "GND" H 2200 4400 50  0000 C CNN
 F 2 "" H 2200 4550 50  0000 C CNN
