File: MoonLander_IO.sch (KiCad schematic (older format))
At the start: 6 parts

Commit message: first whack at layout - unrouted
Parts:
- added SW502: SW_PUSH, GrayCatLabs:PTS810, symbol SW_PUSH
- D501: renamed from D?; footprint (none) -> GrayCatLabs:PLCC4
- P501: renamed from P?; footprint (none) -> GrayCatLabs:Header_2mm_2x8
- R501, R502, R503: renamed from R?; footprint (none) -> Resistors_SMD:R_0402
- SW501: renamed from SW?; footprint (none) -> GrayCatLabs:PTS810
Connections:
- net GND: now also P501.16 (P16), SW502.2; no longer P501.2 (P2)
- net I2C0_SCL: now also P501.1 (P1); no longer P501.3 (P3)
- net I2C0_SDA: now also P501.2 (P2); no longer P501.4 (P4)
- net PIO0_13/ADC_10: now also P501.13 (P13); no longer P501.16 (P16)
- net PIO0_14/ADC_2: now also P501.5 (P5); no longer P501.8 (P8)
- net PIO0_15: now also P501.3 (P3); no longer P501.5 (P5)
- net PIO0_16: now also P501.4 (P4); no longer P501.6 (P6)
- net PIO0_17/ADC_9: now also P501.14 (P14); no longer P501.15 (P15)
- net PIO0_18/ADC_8: now also P501.11 (P11); no longer P501.14 (P14)
- net PIO0_19/ADC_7: now also P501.12 (P12); no longer P501.13 (P13)
- net PIO0_20/ADC_6: now also P501.9 (P9); no longer P501.12 (P12)
- net PIO0_21/ADC_5: now also P501.10 (P10); no longer P501.11 (P11)
- net PIO0_22/ADC_4: now also P501.7 (P7); no longer P501.10 (P10)
- net PIO0_23/ADC_3: now also P501.8 (P8); no longer P501.9 (P9)
- net PIO0_6/ADC_1: now also P501.6 (P6); no longer P501.7 (P7)
- net VCC: now also P501.15 (P15); no longer P501.1 (P1)
- new net RESET: SW502.1
Other:
- moved on the sheet: P501
Changed lines of the file:
@@
 Text HLabel 7100 3800 2    60   BiDi ~ 0
 I2C0_SDA
-Text HLabel 5650 5200 0    60   Input ~ 0
+Text HLabel 5650 5200 0    60   Output ~ 0
 ISP_ENTRY
 $Comp
-L SW_PUSH SW?
+L SW_PUSH SW501
 U 1 1 5660FFA0
 P 6250 5200
-F 0 "SW?" H 6400 5310 50  0000 C CNN
+F 0 "SW501" H 6400 5310 50  0000 C CNN
 F 1 "SW_PUSH" H 6250 5120 50  0000 C CNN
-F 2 "" H 6250 5200 50  0000 C CNN
+F 2 "GrayCatLabs:PTS810" H 6250 5200 50  0001 C CNN
 F 3 "" H 6250 5200 50  0000 C CNN
 	1    6250 5200
 	1    0    0    -1
 $EndComp
-$Comp
-L GND #PWR?
-U 1 1 566103AA
-P 6800 5300
-F 0 "#PWR?" H 6800 5050 50  0001 C CNN
-F 1 "GND" H 6800 5150 50  0000 C CNN
-F 2 "" H 6800 5300 50  0000 C CNN
-F 3 "" H 6800 5300 50  0000 C CNN
-	1    6800 5300
-	1    0    0    -1
-$EndComp
 Text HLabel 5050 2250 0    60   BiDi ~ 0
 LED_R
+Text HLabel 7100 4000 2    60   BiDi ~ 0
+PIO0_6/ADC_1
+Text HLabel 5400 4400 0    60   BiDi ~ 0
+PIO0_13/ADC_10
 Text HLabel 5400 4000 0    60   BiDi ~ 0
-PIO0_6/ADC_1
-Text HLabel 7100 4400 2    60   BiDi ~ 0
-PIO0_13/ADC_10
-Text HLabel 7100 4000 2    60   BiDi ~ 0
 PIO0_14/ADC_2
 Text HLabel 5400 3900 0    60   BiDi ~ 0
@@
 Text HLabel 7100 3900 2    60   BiDi ~ 0
 PIO0_16
-Text HLabel 5400 4400 0    60   BiDi ~ 0
+Text HLabel 7100 4400 2    60   BiDi ~ 0
 PIO0_17/ADC_9
+Text HLabel 5400 4300 0    60   BiDi ~ 0
+PIO0_18/ADC_8
 Text HLabel 7100 4300 2    60   BiDi ~ 0
-PIO0_18/ADC_8
-Text HLabel 5400 4300 0    60   BiDi ~ 0
 PIO0_19/ADC_7
+Text HLabel 5400 4200 0    60   BiDi ~ 0
+PIO0_20/ADC_6
 Text HLabel 7100 4200 2    60   BiDi ~ 0
-PIO0_20/ADC_6
-Text HLabel 5400 4200 0    60   BiDi ~ 0
 PIO0_21/ADC_5
+Text HLabel 5400 4100 0    60   BiDi ~ 0
+PIO0_22/ADC_4
 Text HLabel 7100 4100 2    60   BiDi ~ 0
-PIO0_22/ADC_4
-Text HLabel 5400 4100 0    60   BiDi ~ 0
 PIO0_23/ADC_3
 Text HLabel 5050 2450 0    60   BiDi ~ 0
@@
 LED_B
 $Comp
-L VCC #PWR?
+L VCC #PWR022
 U 1 1 56611529
-P 5200 3450
-F 0 "#PWR?" H 5200 3300 50  0001 C CNN
-F 1 "VCC" H 5200 3600 50  0000 C CNN
-F 2 "" H 5200 3450 50  0000 C CNN
-F 3 "" H 5200 3450 50  0000 C CNN
-	1    5200 3450
-	1    0    0    -1
-$EndComp
-$Comp
-L GND #PWR?
+P 4400 4250
+F 0 "#PWR022" H 4400 4100 50  0001 C CNN
+F 1 "VCC" H 4400 4400 50  0000 C CNN
+F 2 "" H 4400 4250 50  0000 C CNN
+F 3 "" H 4400 4250 50  0000 C CNN
+	1    4400 4250
+	1    0    0    -1
+$EndComp
+$Comp
+L GND #PWR023
 U 1 1 5661153F
-P 8150 3800
-F 0 "#PWR?" H 8150 3550 50  0001 C CNN
-F 1 "GND" H 8150 3650 50  0000 C CNN
-F 2 "" H 8150 3800 50  0000 C CNN
-F 3 "" H 8150 3800 50  0000 C CNN
-	1    8150 3800
-	1    0    0    -1
-$EndComp
-$Comp
-L CONN_02X08 P?
+P 8150 4600
+F 0 "#PWR023" H 8150 4350 50  0001 C CNN
+F 1 "GND" H 8150 4450 50  0000 C CNN
+F 2 "" H 8150 4600 50  0000 C CNN
+F 3 "" H 8150 4600 50  0000 C CNN
+	1    8150 4600
+	1    0    0    -1
+$EndComp
+$Comp
+L CONN_02X08 P501
 U 1 1 566116D3
-P 6250 4050
-F 0 "P?" H 6250 4500 50  0000 C CNN
-F 1 "CONN_02X08" V 6250 4050 50  0000 C CNN
-F 2 "" H 6250 2850 50  0000 C CNN
-F 3 "" H 6250 2850 50  0000 C CNN
-	1    6250 4050
+P 6250 4150
+F 0 "P501" H 6250 4600 50  0000 C CNN
+F 1 "CONN_02X08" V 6250 4150 50  0000 C CNN
+F 2 "GrayCatLabs:Header_2mm_2x8" H 6250 2950 50  0001 C CNN
+F 3 "" H 6250 2950 50  0000 C CNN
+	1    6250 4150
 	1    0    0    -1
 $EndComp
@@
 	6550 5200 6800 5200
 Wire Wire Line
-	6800 5200 6800 5300
+	6800 5200 6800 5900
 Wire Wire Line
 	5650 5200 5950 5200
 Wire Wire Line
-	8150 3700 8150 3800
-Wire Wire Line
-	6500 3700 8150 3700
-Wire Wire Line
-	5200 3450 5200 3700
-Wire Wire Line
-	5200 3700 6000 3700
+	8150 4500 8150 4600
+Wire Wire Line
+	6500 4500 8150 4500
+Wire Wire Line
+	4400 4250 4400 4500
+Wire Wire Line
+	4400 4500 6000 4500
 Wire Wire Line
 	7100 3800 6500 3800
@@
 	6000 3800 5400 3800
 $Comp
-L LED_RABG D?
+L LED_RABG D501
 U 1 1 56611E54
 P 6250 2450
-F 0 "D?" H 6325 2800 50  0000 C CNN
+F 0 "D501" H 6325 2800 50  0000 C CNN
 F 1 "LED_RABG" H 6275 2100 50  0000 C CNN
-F 2 "" H 6200 2400 50  0000 C CNN
+F 2 "GrayCatLabs:PLCC4" H 6200 2400 50  0001 C CNN
 F 3 "" H 6200 2400 50  0000 C CNN
 	1    6250 2450
@@
 $EndComp
 $Comp
-L R R?
+L R R501
 U 1 1 56611F27
 P 5500 2250
-F 0 "R?" V 5580 2250 50  0000 C CNN
+F 0 "R501" V 5580 2250 50  0000 C CNN
 F 1 "R" V 5500 2250 50  0000 C CNN
-F 2 "" V 5430 2250 50  0000 C CNN
+F 2 "Resistors_SMD:R_0402" V 5430 2250 50  0001 C CNN
 F 3 "" H 5500 2250 50  0000 C CNN
 	1    5500 2250
@@
 $EndComp
 $Comp
-L R R?
+L R R502
 U 1 1 56611F94
 P 5500 2450
-F 0 "R?" V 5580 2450 50  0000 C CNN
+F 0 "R502" V 5580 2450 50  0000 C CNN
 F 1 "R" V 5500 2450 50  0000 C CNN
-F 2 "" V 5430 2450 50  0000 C CNN
+F 2 "Resistors_SMD:R_0402" V 5430 2450 50  0001 C CNN
 F 3 "" H 5500 2450 50  0000 C CNN
 	1    5500 2450
@@
 $EndComp
 $Comp
-L R R?
+L R R503
 U 1 1 56611FBC
 P 5500 2650
-F 0 "R?" V 5580 2650 50  0000 C CNN
+F 0 "R503" V 5580 2650 50  0000 C CNN
 F 1 "R" V 5500 2650 50  0000 C CNN
-F 2 "" V 5430 2650 50  0000 C CNN
+F 2 "Resistors_SMD:R_0402" V 5430 2650 50  0001 C CNN
 F 3 "" H 5500 2650 50  0000 C CNN
 	1    5500 2650
@@
 	6950 2150 6950 2450
 $Comp
-L VCC #PWR?
+L VCC #PWR024
 U 1 1 566122B0
 P 6950 2150
-F 0 "#PWR?" H 6950 2000 50  0001 C CNN
+F 0 "#PWR024" H 6950 2000 50  0001 C CNN
 F 1 "VCC" H 6950 2300 50  0000 C CNN
 F 2 "" H 6950 2150 50  0000 C CNN
@@
 Text Notes 5500 3000 0    60   ~ 0
 Cree CLVBA-FKA-CA1D181BB7R3R3
+Text HLabel 5650 5800 0    60   Output ~ 0
+RESET
+$Comp
+L SW_PUSH SW502
+U 1 1 565FFC99
+P 6250 5800
+F 0 "SW502" H 6400 5910 50  0000 C CNN
+F 1 "SW_PUSH" H 6250 5720 50  0000 C CNN
+F 2 "GrayCatLabs:PTS810" H 6250 5800 50  0001 C CNN
+F 3 "" H 6250 5800 50  0000 C CNN
+	1    6250 5800
+	1    0    0    -1
+$EndComp
+$Comp
+L GND #PWR025
+U 1 1 565FFC9F
+P 6800 5900
+F 0 "#PWR025" H 6800 5650 50  0001 C CNN
+F 1 "GND" H 6800 5750 50  0000 C CNN
+F 2 "" H 6800 5900 50  0000 C CNN
+F 3 "" H 6800 5900 50  0000 C CNN
+	1    6800 5900
+	1    0    0    -1
+$EndComp
+Wire Wire Line
+	6800 5800 6550 5800
+Wire Wire Line
+	5650 5800 5950 5800
+Connection ~ 6800 5800
 $EndSCHEMATC

Commit message: simplified 2 layer version
Parts:
- removed D501: LED_RABG, GrayCatLabs:PLCC4, symbol LED_RABG
- removed R501, R502, R503: R, Resistors_SMD:R_0402, symbol R
- added D3: LED, LEDs:LED-0603, symbol LED
- added R5: 470, Resistors_SMD:R_0402, symbol R
- P4: renamed from P501; footprint GrayCatLabs:Header_2mm_2x8 -> GrayCatLabs:Header_2mm_2x6; symbol CONN_02X08 -> CONN_02X07
- renumbered SW501 to SW1, SW502 to SW2
Connections:
- net PIO0_15 is gone; now on net PIO0_14/ADC_2: P4.3 (P3)
- net PIO0_16 is gone; now on net PIO0_6/ADC_1: P4.4 (P4)
- net GND: now also P4.2 (P2), R5.2; no longer P4.16 (P16)
- net I2C0_SCL: now also P4.13 (P13); no longer P4.1 (P1)
- net I2C0_SDA: now also P4.14 (P14); no longer P4.2 (P2)
- net PIO0_13/ADC_10: now also P4.11 (P11); no longer P4.13 (P13)
- net PIO0_14/ADC_2: no longer P4.5 (P5)
- net PIO0_17/ADC_9: now also P4.12 (P12); no longer P4.14 (P14)
- net PIO0_18/ADC_8: now also P4.9 (P9); no longer P4.11 (P11)
- net PIO0_19/ADC_7: now also P4.10 (P10); no longer P4.12 (P12)
- net PIO0_20/ADC_6: now also P4.7 (P7); no longer P4.9 (P9)
- net PIO0_21/ADC_5: now also P4.8 (P8); no longer P4.10 (P10)
- net PIO0_22/ADC_4: now also P4.5 (P5); no longer P4.7 (P7)
- net PIO0_23/ADC_3: now also P4.6 (P6); no longer P4.8 (P8)
- net PIO0_6/ADC_1: no longer P4.6 (P6)
- net VCC: now also P4.1 (P1); no longer P4.15 (P15)
- new net: D3.1 (K), R5.1
- new net LED: D3.2 (A)
Other:
- note removed: "Cree CLVBA-FKA-CA1D181BB7R3R3"
- moved on the sheet: SW1, SW2
